File: rde-board-v2.0/rde-board-v2.0.kicad_pcb (KiCad board)
At the start: 2 copper layers, 56 x 65 mm, 19 parts, among them J1 RPI conn, J2 Mouse / Joy 1, J3 Joy 2, U1 ULN2003A, U2 ULN2003A

Commit message: Update rde-board
Parts:
- added REF**: OSHW-Logo2_7.3x6mm_SilkScreen, Symbol:OSHW-Logo2_7.3x6mm_SilkScreen, B.Cu at (130.5, 110.3)
- added REF**: KiCad-Logo2_5mm_SilkScreen, Symbol:KiCad-Logo2_5mm_SilkScreen, B.Cu at (142.8, 109.9)
Other:
- board text added: "RetroDevEm v2.0"
